File: minirouter/minirouter.kicad_sch (KiCad schematic)
At the start: 1 part

Commit message: added lib stuff
Other:
- removed sheet ETHERNET
- removed sheet PCIE
- removed sheet USB
- moved on the sheet: Module1A, Module1B
Changed lines of the file:
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@@
 	(symbol
 		(lib_id "CM4IO:ComputeModule4-CM4")
-		(at 71.12 121.92 0)
+		(at 147.32 81.28 0)
 		(unit 1)
 		(exclude_from_sim no)
@@
 		(fields_autoplaced yes)
 		(property "Reference" "Module1"
-			(at 68.58 53.34 0)
+			(at 144.78 12.7 0)
 			(effects
 				(font
@@
 		)
 		(property "Value" "ComputeModule4-CM4"
-			(at 68.58 55.88 0)
+			(at 144.78 15.24 0)
 			(effects
 				(font
@@
 		)
 		(property "Footprint" "router-footprints:Raspberry-Pi-4-Compute-Module"
-			(at 213.36 148.59 0)
+			(at 289.56 107.95 0)
 			(effects
 				(font
@@
 		)
 		(property "Datasheet" ""
-			(at 213.36 148.59 0)
+			(at 289.56 107.95 0)
 			(effects
 				(font
@@
 		)
 		(property "Description" ""
-			(at 71.12 121.92 0)
+			(at 147.32 81.28 0)
 			(effects
 				(font
@@
 		)
 		(property "Field4" "Hirose"
-			(at 68.58 58.42 0)
+			(at 144.78 17.78 0)
 			(effects
 				(font
@@
 		)
 		(property "Field5" "2x DF40C-100DS-0.4V"
-			(at 68.58 60.96 0)
+			(at 144.78 20.32 0)
 			(effects
 				(font
@@
 	(symbol
 		(lib_id "CM4IO:ComputeModule4-CM4")
-		(at 86.36 123.19 0)
+		(at 77.47 86.36 0)
 		(unit 2)
 		(exclude_from_sim no)
@@
 		(fields_autoplaced yes)
 		(property "Reference" "Module1"
-			(at 226.06 49.53 0)
+			(at 217.17 12.7 0)
 			(effects
 				(font
@@
 		)
 		(property "Value" "ComputeModule4-CM4"
-			(at 226.06 52.07 0)
+			(at 217.17 15.24 0)
 			(effects
 				(font
@@
 		)
 		(property "Footprint" "router-footprints:Raspberry-Pi-4-Compute-Module"
-			(at 228.6 149.86 0)
+			(at 219.71 113.03 0)
 			(effects
 				(font
@@
 		)
 		(property "Datasheet" ""
-			(at 228.6 149.86 0)
+			(at 219.71 113.03 0)
 			(effects
 				(font
@@
 		)
 		(property "Description" ""
-			(at 86.36 123.19 0)
+			(at 77.47 86.36 0)
 			(effects
 				(font
@@
 		)
 		(property "Field4" "Hirose"
-			(at 226.06 54.61 0)
+			(at 217.17 17.78 0)
 			(effects
 				(font
@@
 		)
 		(property "Field5" "2x DF40C-100DS-0.4V"
-			(at 226.06 57.15 0)
+			(at 217.17 20.32 0)
 			(effects
 				(font
@@
 				)
 			)
-		)
-	)
-	(sheet
-		(at 326.39 60.96)
-		(size 41.91 41.91)
-		(exclude_from_sim no)
-		(in_bom yes)
-		(on_board yes)
-		(dnp no)
-		(fields_autoplaced yes)
-		(stroke
-			(width 0.1524)
-			(type solid)
-		)
-		(fill
-			(color 0 0 0 0.0000)
-		)
-		(property "Sheetname" "USB"
-			(at 326.39 60.2484 0)
-			(effects
-				(font
-					(size 1.27 1.27)
-				)
-				(justify left bottom)
-			)
-		)
-		(property "Sheetfile" "usb.kicad_sch"
-			(at 326.39 103.4546 0)
-			(effects
-				(font
-					(size 1.27 1.27)
-				)
-				(justify left top)
-			)
-		)
-		(instances
-			(project "minirouter"
-				(path "/ed318ed4-4a6b-4ca2-a636-0816a30f875c"
-					(page "2")
-				)
-			)
-		)
-	)
-	(sheet
-		(at 326.39 184.15)
-		(size 43.18 66.04)
-		(exclude_from_sim no)
-		(in_bom yes)
-		(on_board yes)
-		(dnp no)
-		(fields_autoplaced yes)
-		(stroke
-			(width 0.1524)
-			(type solid)
-		)
-		(fill
-			(color 0 0 0 0.0000)
-		)
-		(property "Sheetname" "PCIE"
-			(at 326.39 183.4384 0)
-			(effects
-				(font
-					(size 1.27 1.27)
-				)
-				(justify left bottom)
-			)
-		)
-		(property "Sheetfile" "pcie.kicad_sch"
-			(at 326.39 250.7746 0)
-			(effects
-				(font
-					(size 1.27 1.27)
-				)
-				(justify left top)
-			)
-		)
-		(instances
-			(project "minirouter"
-				(path "/ed318ed4-4a6b-4ca2-a636-0816a30f875c"
-					(page "4")
-				)
-			)
-		)
-	)
-	(sheet
-		(at 326.39 110.49)
-		(size 41.91 64.77)
-		(exclude_from_sim no)
-		(in_bom yes)
-		(on_board yes)
-		(dnp no)
-		(fields_autoplaced yes)
-		(stroke
-			(width 0.1524)
-			(type solid)
-		)
-		(fill
-			(color 0 0 0 0.0000)
-		)
-		(property "Sheetname" "ETHERNET"
-			(at 326.39 109.7784 0)
-			(effects
-				(font
-					(size 1.27 1.27)
-				)
-				(justify left bottom)
-			)
-		)
-		(property "Sheetfile" "ethernet.kicad_sch"
-			(at 326.39 175.8446 0)
-			(effects
-				(font
-					(size 1.27 1.27)
-				)
-				(justify left top)
-			)
-		)
-		(instances
-			(project "minirouter"
-				(path "/ed318ed4-4a6b-4ca2-a636-0816a30f875c"
-					(page "3")
-				)
-			)
